Commit message: basic_robot xacro files update

File: src/basic_robot/Models/basic_robot.urdf.xacro (robot description, xacro)
@@ -2,3 +2,4 @@
 <robot xmlns:xacro="http://www.ros.org/wiki/xacro"  name="basic_robot">
     <xacro:include filename="basic_robot_core.xacro"/>
+    <xacro:include filename="gazebo_control.xacro"/>
 </robot>

File: src/basic_robot/Models/basic_robot_core.xacro (robot description, xacro)
@@ -33,4 +33,7 @@
         </xacro:inertial_box>
     </link>
+    <gazebo reference="chassis">
+        <material>Gazebo/White</material>
+    </gazebo>
     <!--Left Wheel Link-->
     <joint name="left_wheel_joint" type="continuous">
@@ -56,4 +59,7 @@
         </xacro:inertial_cylinder>
     </link>
+    <gazebo reference="left_wheel">
+        <material>Gazebo/Blue</material>
+    </gazebo>
     <!--Right Wheel Link-->
     <joint name="right_wheel_joint" type="continuous">
@@ -79,4 +85,7 @@
         </xacro:inertial_cylinder>
     </link>
+    <gazebo reference="right_wheel">
+        <material>Gazebo/Blue</material>
+    </gazebo>
     <!--Caster Wheel-->
     <joint name="caster_wheel_joint" type="fixed">
@@ -101,3 +110,6 @@
         </xacro:inertial_sphere>
     </link>
+    <gazebo reference="caster_wheel">
+        <material>Gazebo/Black</material>
+    </gazebo>
 </robot>

Commit message: Changes to .xarco

File: src/basic_robot/Models/basic_robot.urdf.xacro (robot description, xacro)
@@ -1,5 +1,5 @@
 <?xml version="1.0"?>
-<robot xmlns:xacro="http://www.ros.org/wiki/xacro"  name="basic_robot">
-    <xacro:include filename="basic_robot_core.xacro"/>
-    <xacro:include filename="gazebo_control.xacro"/>
+<robot xmlns:xacro="http://www.ros.org/wiki/xacro"  name="robot">
+    <xacro:include filename="basic_robot_core.xacro" />
+    <xacro:include filename="gazebo_control.xacro" />
 </robot>

File: src/basic_robot/Models/basic_robot_core.xacro (robot description, xacro)
@@ -6,5 +6,5 @@
     <link name="base_link">
     </link>
-    <!--Chassis Link-->
+<!-- CHASSIS LINK -->
     <joint name="chassis_joint" type="fixed">
         <parent link="base_link"/>
@@ -29,6 +29,6 @@
             </geometry>
         </collision>
-        <xacro:inertial_box mass="0.5"  x="0.3" y="0.3" z="0.15">
-            <origin xyz="0.15 0 0.075"  rpy="0 0 0"/>
+        <xacro:inertial_box mass="0.5" x="0.3" y="0.3" z="0.15">
+            <origin xyz="0.15 0 0.075" rpy="0 0 0"/>
         </xacro:inertial_box>
     </link>
@@ -36,9 +36,9 @@
         <material>Gazebo/White</material>
     </gazebo>
-    <!--Left Wheel Link-->
+    <!-- LEFT WHEEL LINK -->
     <joint name="left_wheel_joint" type="continuous">
         <parent link="base_link"/>
         <child link="left_wheel"/>
-        <origin xyz="0.0 0.175 0.0" rpy="-${pi/2} 0 0"/>
+        <origin xyz="0 0.175 0" rpy="-${pi/2} 0 0" />
         <axis xyz="0 0 1"/>
     </joint>
@@ -55,5 +55,5 @@
             </geometry>
         </collision>
-        <xacro:inertial_cylinder    mass="0.1"  length="0.04"   radius="0.05">
+        <xacro:inertial_cylinder mass="0.1" length="0.04" radius="0.05">
             <origin xyz="0 0 0" rpy="0 0 0"/>
         </xacro:inertial_cylinder>
@@ -62,9 +62,9 @@
         <material>Gazebo/Blue</material>
     </gazebo>
-    <!--Right Wheel Link-->
+    <!-- RIGHT WHEEL LINK -->
     <joint name="right_wheel_joint" type="continuous">
         <parent link="base_link"/>
         <child link="right_wheel"/>
-        <origin xyz="0.0 -0.175 0.0" rpy="${pi/2} 0 0"/>
+        <origin xyz="0 -0.175 0" rpy="${pi/2} 0 0" />
         <axis xyz="0 0 -1"/>
     </joint>
@@ -81,5 +81,5 @@
             </geometry>
         </collision>
-        <xacro:inertial_cylinder    mass="0.1"  length="0.04"   radius="0.05">
+        <xacro:inertial_cylinder mass="0.1" length="0.04" radius="0.05">
             <origin xyz="0 0 0" rpy="0 0 0"/>
         </xacro:inertial_cylinder>
@@ -88,5 +88,5 @@
         <material>Gazebo/Blue</material>
     </gazebo>
-    <!--Caster Wheel-->
+    <!-- CASTER WHEEL LINK -->
     <joint name="caster_wheel_joint" type="fixed">
         <parent link="chassis"/>
@@ -106,5 +106,5 @@
             </geometry>
         </collision>
-        <xacro:inertial_sphere mass="0.1"   radius="0.05">
+        <xacro:inertial_sphere mass="0.1" radius="0.05">
             <origin xyz="0 0 0" rpy="0 0 0"/>
         </xacro:inertial_sphere>
@@ -112,4 +112,6 @@
     <gazebo reference="caster_wheel">
         <material>Gazebo/Black</material>
+        <mu1 value="0.001"/>
+        <mu2 value="0.001"/>
     </gazebo>
 </robot>

File: src/basic_robot/Models/gazebo_control.xacro (robot description, xacro)
@@ -2,16 +2,16 @@
 <robot xmlns:xacro="http://www.ros.org/wiki/xacro">
     <gazebo>
-        <plugin name="diff_drive"   filename="libgazebo_ros_diff_drive.so">
-           <!--Wheel Info-->
+        <plugin name="diff_drive" filename="libgazebo_ros_diff_drive.so">
+            <!-- Wheel Information -->
             <left_joint>left_wheel_joint</left_joint>
             <right_joint>right_wheel_joint</right_joint>
             <wheel_separation>0.35</wheel_separation>
             <wheel_diameter>0.1</wheel_diameter>
-            <!--Limits-->
+            <!-- Limits -->
             <max_wheel_torque>200</max_wheel_torque>
             <max_wheel_acceleration>10.0</max_wheel_acceleration>
-            <!--Output-->
+            <!-- Output -->
+            <robot_base_frame>base_link</robot_base_frame>
             <odometry_frame>odom</odometry_frame>
-            <robot_base_frame>base_link</robot_base_frame>
             <publish_odom>true</publish_odom>
             <publish_odom_tf>true</publish_odom_tf>
