Commit message: Changing link name to make use of slam_toolbox for mapping

File: src/basic_robot/Models/basic_robot_core.xacro (robot description, xacro)
@@ -4,9 +4,9 @@
     <xacro:include filename="inertial_macros.xacro"/>
     <!--Base Link-->
-    <link name="base_link">
+    <link name="base_footprint">
     </link>
 <!-- CHASSIS LINK -->
     <joint name="chassis_joint" type="fixed">
-        <parent link="base_link"/>
+        <parent link="base_footprint"/>
         <child link="chassis"/>
         <!--origin is on the wheel drive-->
@@ -38,5 +38,5 @@
     <!-- LEFT WHEEL LINK -->
     <joint name="left_wheel_joint" type="continuous">
-        <parent link="base_link"/>
+        <parent link="base_footprint"/>
         <child link="left_wheel"/>
         <origin xyz="0 0.175 0" rpy="-${pi/2} 0 0" />
@@ -64,5 +64,5 @@
     <!-- RIGHT WHEEL LINK -->
     <joint name="right_wheel_joint" type="continuous">
-        <parent link="base_link"/>
+        <parent link="base_footprint"/>
         <child link="right_wheel"/>
         <origin xyz="0 -0.175 0" rpy="${pi/2} 0 0" />

File: src/basic_robot/Models/gazebo_control.xacro (robot description, xacro)
@@ -12,5 +12,5 @@
             <max_wheel_acceleration>10.0</max_wheel_acceleration>
             <!-- Output -->
-            <robot_base_frame>base_link</robot_base_frame>
+            <robot_base_frame>base_footprint</robot_base_frame>
             <odometry_frame>odom</odometry_frame>
             <publish_odom>true</publish_odom>
